Commit message: Unicos cambios significativos en el archivo summit.urdf.xacro. Habia errores en los controladores de las ruedas porque tambien tenian que tener el tag <hardwareInterface>. Ademas, como advertencia hemos añadido 'hardware_interface/' en el tag de <join> ya que recomendaba.

File: summit_description/urdf/summit.urdf.xacro (robot description, xacro)
@@ -81,5 +81,5 @@
     <visual>
        <!-- visual origin is defined w.r.t. link local coordinate system -->
-       <origin xyz="0 0 0" rpy="0 0 1.5708" />
+       <origin xyz="0 0 0" rpy="0 0 0" />
        <geometry>
          <cylinder radius="0.015" length="0.025"/>
@@ -105,7 +105,9 @@
   <transmission name="joint_blw_trans_dir">
 	<type>transmission_interface/SimpleTransmission</type>
-    <joint name="joint_back_left_wheel_dir" />
+    <joint name="joint_back_left_wheel_dir">
+      <hardwareInterface>hardware_interface/EffortJointInterface</hardwareInterface>
+    </joint>
     <actuator name="joint_blw_motor_dir">
-	  <hardwareInterface>EffortJointInterface</hardwareInterface>
+	    <hardwareInterface>EffortJointInterface</hardwareInterface>
       <mechanicalReduction>${steer_mechanical_reduction}</mechanicalReduction>
 	  <!-- motorTorqueConstant>1</motorTorqueConstant -->
@@ -145,9 +147,11 @@
   <transmission name="joint_blw_trans">
 	 <type>transmission_interface/SimpleTransmission</type>
-     <joint name="joint_back_left_wheel" />
+     <joint name="joint_back_left_wheel">
+       <hardwareInterface>hardware_interface/VelocityJointInterface</hardwareInterface>
+     </joint>
      <actuator name="joint_blw_motor">
 	    <hardwareInterface>VelocityJointInterface</hardwareInterface>
         <mechanicalReduction>${wheel_mechanical_reduction}</mechanicalReduction>
-     	<!-- motorTorqueConstant>1</motorTorqueConstant -->
+     	<!--motorTorqueConstant>1</motorTorqueConstant-->
 	 </actuator>
   </transmission>
@@ -186,5 +190,7 @@
   <transmission name="joint_brw_trans_dir">
 	<type>transmission_interface/SimpleTransmission</type>
-    <joint name="joint_back_right_wheel_dir" />
+    <joint name="joint_back_right_wheel_dir">
+      <hardwareInterface>hardware_interface/EffortJointInterface</hardwareInterface>
+    </joint>
     <actuator name="joint_brw_motor_dir">
 	  <hardwareInterface>EffortJointInterface</hardwareInterface>
@@ -226,5 +232,7 @@
   <transmission name="joint_brw_trans">
 	 <type>transmission_interface/SimpleTransmission</type>
-     <joint name="joint_back_right_wheel" />
+     <joint name="joint_back_right_wheel">
+       <hardwareInterface>hardware_interface/VelocityJointInterface</hardwareInterface>
+     </joint>
      <actuator name="joint_brw_motor">
 	    <hardwareInterface>VelocityJointInterface</hardwareInterface>
@@ -267,5 +275,7 @@
   <transmission name="joint_flw_trans_dir">
 	<type>transmission_interface/SimpleTransmission</type>
-    <joint name="joint_front_left_wheel_dir" />
+    <joint name="joint_front_left_wheel_dir">
+      <hardwareInterface>hardware_interface/EffortJointInterface</hardwareInterface>
+    </joint>
     <actuator name="joint_flw_motor_dir">
 	  <hardwareInterface>EffortJointInterface</hardwareInterface>
@@ -307,5 +317,7 @@
   <transmission name="joint_flw_trans">
 	 <type>transmission_interface/SimpleTransmission</type>
-     <joint name="joint_front_left_wheel" />
+     <joint name="joint_front_left_wheel">
+       <hardwareInterface>hardware_interface/VelocityJointInterface</hardwareInterface>
+     </joint>
      <actuator name="joint_flw_motor">
 	    <hardwareInterface>VelocityJointInterface</hardwareInterface>
@@ -348,5 +360,7 @@
   <transmission name="joint_frw_trans_dir">
 	<type>transmission_interface/SimpleTransmission</type>
-    <joint name="joint_front_right_wheel_dir" />
+    <joint name="joint_front_right_wheel_dir">
+      <hardwareInterface>hardware_interface/EffortJointInterface</hardwareInterface>
+    </joint>
     <actuator name="joint_frw_motor_dir">
 	  <hardwareInterface>EffortJointInterface</hardwareInterface>
@@ -388,5 +402,7 @@
   <transmission name="joint_frw_trans">
 	 <type>transmission_interface/SimpleTransmission</type>
-     <joint name="joint_front_right_wheel" />
+     <joint name="joint_front_right_wheel">
+       <hardwareInterface>hardware_interface/VelocityJointInterface</hardwareInterface>
+     </joint>
      <actuator name="joint_frw_motor">
 	    <hardwareInterface>VelocityJointInterface</hardwareInterface>
@@ -479,5 +495,7 @@
   <transmission name="joint_pan_trans">
 	 <type>transmission_interface/SimpleTransmission</type>
-     <joint name="joint_camera_pan" />
+     <joint name="joint_camera_pan">
+       <hardwareInterface>hardware_interface/EffortJointInterface</hardwareInterface>
+     </joint>
      <actuator name="pan_motor">
 	   <hardwareInterface>EffortJointInterface</hardwareInterface>
@@ -503,5 +521,7 @@
   <transmission name="joint_tilt_trans">
 	 <type>transmission_interface/SimpleTransmission</type>
-     <joint name="joint_camera_tilt" />
+     <joint name="joint_camera_tilt">
+       <hardwareInterface>hardware_interface/EffortJointInterface</hardwareInterface>
+     </joint>
      <actuator name="tilt_motor">
 	   <hardwareInterface>EffortJointInterface</hardwareInterface>

Commit message: He colocado la camara kinect. He cambiado los nodos para que publique el de la camara. He modificado los archivos del urdf para que se vea la camara kinect. He recolocado la camara kinect para que no aparezca en el suelo.

File: summit_description/urdf/summit.urdf.xacro (robot description, xacro)
@@ -24,4 +24,10 @@
   <xacro:property name="ptz_joint_damping" value="0.1" />
   <xacro:property name="ptz_mechanical_reduction" value="1.0" />
+  <xacro:property name="cam_px" value="-0.087" />
+	<xacro:property name="cam_py" value="-0.0125" />
+	<xacro:property name="cam_pz" value="0.2870" />
+	<xacro:property name="cam_or" value="0" />
+	<xacro:property name="cam_op" value="0" />
+  <xacro:property name="cam_oy" value="0" />
   <!-- BASE FOOTPRINT -->
   <!-- base_footprint is a fictitious link(frame) that is on the ground right below base_link origin,
@@ -463,4 +469,91 @@
       </collision>
   </link>
+  <!-- KINECT SENSOR -->
+  <joint name="kinect_rgb_joint" type="fixed">
+      <origin xyz="0.10 0 0.2825" rpy="0 0 0"/>
+      <parent link="base_link"/>
+      <child link="kinect_rgb_base_link" />
+    </joint>
+    <link name="kinect_rgb_base_link">
+      <inertial>
+        <mass value="0.001" />
+        <origin xyz="0 0 0" />
+        <inertia ixx="0.0001" ixy="0.0" ixz="0.0"
+                 iyy="0.0001" iyz="0.0"
+                 izz="0.0001" />
+      </inertial>
+    </link>
+    <joint name="kinect_rgb_optical_joint" type="fixed">
+      <origin xyz="0 0 0" rpy="${-PI/2} 0 ${-PI/2}" />
+      <parent link="kinect_rgb_base_link" />
+      <child link="kinect_rgb_optical_link" />
+    </joint>
+    <link name="kinect_rgb_optical_link">
+      <inertial>
+        <mass value="0.001" />
+        <origin xyz="0 0 0" />
+        <inertia ixx="0.0001" ixy="0.0" ixz="0.0"
+                 iyy="0.0001" iyz="0.0"
+                 izz="0.0001" />
+      </inertial>
+    </link>
+  <joint name="kinect_joint" type="fixed">
+    <origin xyz="-0.031 ${-cam_py} -0.016" rpy="0 0 0"/>
+    <parent link="kinect_rgb_base_link"/>
+    <child link="kinect_link"/>
+  </joint>
+    <link name="kinect_link">
+    <visual>
+     <origin xyz="0 0 0" rpy="0 0 ${PI/2}"/>
+      <geometry>
+       <mesh filename="package://robotnik_sensors/meshes/kinect.dae"/>
+      </geometry>
+    </visual>
+	  <collision>
+      <origin xyz="0.0 0.0 0.0" rpy="0 0 0"/>
+	    <geometry>
+	      <box size="0.07271 0.27794 0.073"/>
+	    </geometry>
+	  </collision>
+    <inertial>
+      <mass value="0.001" />
+      <origin xyz="0 0 0" />
+      <inertia ixx="0.0001" ixy="0.0" ixz="0.0"
+               iyy="0.0001" iyz="0.0"
+               izz="0.0001" />
+    </inertial>
+  </link>
+  <!-- The fixed joints & links below are usually published by static_transformers launched by the OpenNi launch
+       files. However, for Gazebo simulation we need them, so we add them here.
+       (Hence, don't publish them additionally!) -->
+	<joint name="kinect_depth_joint" type="fixed">
+	  <origin xyz="0 ${2 * -cam_py} 0" rpy="0 0 0" />
+	  <parent link="kinect_rgb_base_link" />
+	  <child link="kinect_depth_link" />
+	</joint>
+	<link name="kinect_depth_link">
+    <inertial>
+      <mass value="0.001" />
+      <origin xyz="0 0 0" />
+      <inertia ixx="0.0001" ixy="0.0" ixz="0.0"
+               iyy="0.0001" iyz="0.0"
+               izz="0.0001" />
+    </inertial>
+	</link>
+	<joint name="kinect_depth_optical_joint" type="fixed">
+	  <origin xyz="0 0 0" rpy="${-PI/2} 0 ${-PI/2}" />
+	  <parent link="kinect_depth_link" />
+	  <child link="kinect_depth_optical_link" />
+	</joint>
+	<link name="kinect_depth_optical_link">
+    <inertial>
+      <mass value="0.001" />
+      <origin xyz="0 0 0" />
+      <inertia ixx="0.0001" ixy="0.0" ixz="0.0"
+               iyy="0.0001" iyz="0.0"
+               izz="0.0001" />
+    </inertial>
+	</link>
+  <!--     -->
   <!-- AXIS PTZ CAMERA WITH PAN AND TILT -->
   <link name="camera_base_link">

Commit message: Hemos quitado los sensores de hokuyo y camera, hemos añadido los del kinect y ademas renombrado kinect por camera y link por frames para futuro.

File: summit_description/urdf/summit.urdf.xacro (robot description, xacro)
@@ -417,30 +417,4 @@
 	 </actuator>
   </transmission>
-  <!-- HOKUYO SENSOR -->
-  <joint name="hokuyo_laser_joint" type="fixed">
-     <axis xyz="0 1 0" />
-     <origin xyz="0.226 0 0.120"/>
-     <parent link="base_link"/>
-     <child link="hokuyo_laser_link"/>
-  </joint>
-  <link name="hokuyo_laser_link" type="laser">
-    <collision>
-      <origin xyz="0 0 0" rpy="0 0 0"/>
-      <geometry>
-	     <box size="0.1 0.1 0.1"/>
-      </geometry>
-    </collision>
-    <visual>
-      <origin xyz="0 0 0" rpy="0 0 0"/>
-      <geometry>
-        <mesh filename="package://summit_description/meshes/hokuyo-utm30-lx.dae"/>
-      </geometry>
-    </visual>
-    <inertial>
-      <mass value="1e-5" />
-      <origin xyz="0 0 0" rpy="0 0 0"/>
-      <inertia ixx="1e-6" ixy="0" ixz="0" iyy="1e-6" iyz="0" izz="1e-6" />
-    </inertial>
-  </link>
   <!-- IMU SENSOR -->
   <joint name="imu_joint" type="fixed">
@@ -473,7 +447,7 @@
       <origin xyz="0.10 0 0.2825" rpy="0 0 0"/>
       <parent link="base_link"/>
-      <child link="kinect_rgb_base_link" />
+      <child link="camera_rgb_base_frame" />
     </joint>
-    <link name="kinect_rgb_base_link">
+    <link name="camera_rgb_base_frame">
       <inertial>
         <mass value="0.001" />
@@ -486,8 +460,8 @@
     <joint name="kinect_rgb_optical_joint" type="fixed">
       <origin xyz="0 0 0" rpy="${-PI/2} 0 ${-PI/2}" />
-      <parent link="kinect_rgb_base_link" />
-      <child link="kinect_rgb_optical_link" />
+      <parent link="camera_rgb_base_frame" />
+      <child link="camera_rgb_optical_frame" />
     </joint>
-    <link name="kinect_rgb_optical_link">
+    <link name="camera_rgb_optical_frame">
       <inertial>
         <mass value="0.001" />
@@ -500,8 +474,8 @@
   <joint name="kinect_joint" type="fixed">
     <origin xyz="-0.031 ${-cam_py} -0.016" rpy="0 0 0"/>
-    <parent link="kinect_rgb_base_link"/>
-    <child link="kinect_link"/>
-  </joint>
-    <link name="kinect_link">
+    <parent link="camera_rgb_base_frame"/>
+    <child link="camera_link"/>
+  </joint>
+    <link name="camera_link">
     <visual>
      <origin xyz="0 0 0" rpy="0 0 ${PI/2}"/>
@@ -529,8 +503,8 @@
 	<joint name="kinect_depth_joint" type="fixed">
 	  <origin xyz="0 ${2 * -cam_py} 0" rpy="0 0 0" />
-	  <parent link="kinect_rgb_base_link" />
-	  <child link="kinect_depth_link" />
+	  <parent link="camera_rgb_base_frame" />
+	  <child link="camera_depth_frame" />
 	</joint>
-	<link name="kinect_depth_link">
+	<link name="camera_depth_frame">
     <inertial>
       <mass value="0.001" />
@@ -543,8 +517,8 @@
 	<joint name="kinect_depth_optical_joint" type="fixed">
 	  <origin xyz="0 0 0" rpy="${-PI/2} 0 ${-PI/2}" />
-	  <parent link="kinect_depth_link" />
-	  <child link="kinect_depth_optical_link" />
+	  <parent link="camera_depth_frame" />
+	  <child link="camera_depth_optical_frame" />
 	</joint>
-	<link name="kinect_depth_optical_link">
+	<link name="camera_depth_optical_frame">
     <inertial>
       <mass value="0.001" />
@@ -555,70 +529,3 @@
     </inertial>
 	</link>
-  <!--     -->
-  <!-- AXIS PTZ CAMERA WITH PAN AND TILT -->
-  <link name="camera_base_link">
-     <inertial>
-       <mass value="0.1" />
-       <origin xyz="0 0 0" rpy="0 0 0" />
-       <inertia ixx="0.1" ixy="0" ixz="0" iyy="0.1" iyz="0" izz="0.1" />
-    </inertial>
-  </link>
-  <joint name="joint_camera" type="fixed">
-     <axis xyz="0 1 0" />
-     <!--origin xyz="0.180 0.0 0.270"/-->
-     <origin xyz="0.150 0.0 0.240"/>
-     <parent link="base_link"/>
-     <child link="camera_base_link"/>
-  </joint>
-  <link name="camera_pan_link">
-     <inertial>
-       <mass value="0.1" />
-       <origin xyz="0 0 0" rpy="0 0 0" />
-       <inertia ixx="0.1" ixy="0" ixz="0" iyy="0.1" iyz="0" izz="0.1" />
-    </inertial>
-  </link>
-  <joint name="joint_camera_pan" type="continuous">
-     <axis xyz="0 0 1" />
-     <origin xyz="0.0 0.0 0.0"/>
-     <parent link="camera_base_link"/>
-     <child link="camera_pan_link"/>
-     <limit effort="${ptz_joint_effort_limit}" velocity="${ptz_joint_velocity_limit}" lower="-3.1416" upper="3.1416"/>
-     <joint_properties damping="${ptz_joint_damping}" friction="{ptz_joint_friction}"/>
-  </joint>
-  <transmission name="joint_pan_trans">
-	 <type>transmission_interface/SimpleTransmission</type>
-     <joint name="joint_camera_pan">
-       <hardwareInterface>hardware_interface/EffortJointInterface</hardwareInterface>
-     </joint>
-     <actuator name="pan_motor">
-	   <hardwareInterface>EffortJointInterface</hardwareInterface>
-       <mechanicalReduction>${ptz_mechanical_reduction}</mechanicalReduction>
-     </actuator>
-  </transmission>
-  <link name="camera_tilt_link">
-     <inertial>
-       <mass value="0.1" />
-       <!-- origin xyz="0 0 0" rpy="0 0 0" / -->
-       <origin xyz="0 0 0.3" rpy="0 0 0" />
-       <inertia ixx="0.1" ixy="0" ixz="0" iyy="0.1" iyz="0" izz="0.1" />
-    </inertial>
-  </link>
-  <joint name="joint_camera_tilt" type="continuous">
-     <axis xyz="0 1 0" />
-     <origin xyz="0.0 0.0 0.0"/>
-     <parent link="camera_pan_link"/>
-     <child link="camera_tilt_link"/>
-     <limit effort="${ptz_joint_effort_limit}" velocity="${ptz_joint_velocity_limit}" lower="-1.5708" upper="1.5708"/>
-     <joint_properties damping="${ptz_joint_damping}" friction="{ptz_joint_friction}"/>
-  </joint>
-  <transmission name="joint_tilt_trans">
-	 <type>transmission_interface/SimpleTransmission</type>
-     <joint name="joint_camera_tilt">
-       <hardwareInterface>hardware_interface/EffortJointInterface</hardwareInterface>
-     </joint>
-     <actuator name="tilt_motor">
-	   <hardwareInterface>EffortJointInterface</hardwareInterface>
-       <mechanicalReduction>${ptz_mechanical_reduction}</mechanicalReduction>
-     </actuator>
-  </transmission>
 </robot>
